Commit message: Revert urdf to last master branch commit

File: reflex_visualizer/urdf/full_reflex_model.urdf.xacro (robot description, xacro)
@@ -4,25 +4,25 @@
 <!-- ################ XACRO PORTION OF THE URDF, FOR MAKING THE FLEXIBLE JOINTS ################ -->
 <!-- ################ ################ ################ ################ ################ ################ -->
-  <xacro:property name="flex_length" value="0.016" />
-  <xacro:property name="num_steps" value="9" />
-  <xacro:property name="prox_length" value="0.060" />
-  <xacro:property name="pi" value="3.1415" />
-  <xacro:macro name="base_color">
-    <color rgba="0.1 0.1 0.1 1"/>
-  </xacro:macro>
-  <xacro:macro name="swivel_color">
-    <color rgba="0.1 0.1 0.1 1"/>
-  </xacro:macro>
-  <xacro:macro name="proximal_color">
-    <color rgba="0.16 0.16 0.16 1"/>
-  </xacro:macro>
-   <xacro:macro name="distal_color">
-    <color rgba="0.16 0.16 0.16 1"/>
-  </xacro:macro>
-  <xacro:macro name="flex_color">
-    <color rgba="0.2 0.2 .2 1"/>
-  </xacro:macro>
+	<xacro:property name="flex_length" value="0.016" />
+	<xacro:property name="num_steps" value="9" />
+	<xacro:property name="prox_length" value="0.060" />
+	<xacro:property name="pi" value="3.1415" />
+ 	<xacro:macro name="base_color">
+ 		<color rgba="0.1 0.1 0.1 1"/>
+ 	</xacro:macro>
+ 	<xacro:macro name="swivel_color">
+ 		<color rgba="0.1 0.1 0.1 1"/>
+ 	</xacro:macro>
+ 	<xacro:macro name="proximal_color">
+ 		<color rgba="0.16 0.16 0.16 1"/>
+ 	</xacro:macro>
+ 	 <xacro:macro name="distal_color">
+ 		<color rgba="0.16 0.16 0.16 1"/>
+ 	</xacro:macro>
+ 	<xacro:macro name="flex_color">
+ 		<color rgba="0.2 0.2 .2 1"/>
+ 	</xacro:macro>
   <xacro:macro name="pad_color">
-    <color rgba="0.2 0.8 0.75 1"/>
+    <color rgba="0.106 0.227 0.631 1"/>
   </xacro:macro>
   <!-- Macro to make each part of the link -->
@@ -32,5 +32,5 @@
       <visual>
         <origin
-          xyz="0 -0.008 0.001"
+          xyz="0.001 -0.007 0.003"
           rpy="${pi/2} 0 ${pi/2}" />
         <geometry>
@@ -44,123 +44,83 @@
       </visual>
     </link>
-    <link name="finger[${finger_id}]/flex_link[${flex_id}]/virtual_link[1]"/>
-    <link name="finger[${finger_id}]/flex_link[${flex_id}]/virtual_link[2]"/>
   </xacro:macro>
-  <!-- Macro to one flex body link to the next -->
-  <xacro:macro name="flex_joint" params="finger_id link_parent link_child">
-    <joint name="finger[${finger_id}]/flex_link[${link_parent}]/flex_joint_from_flex_link[${link_parent}]_to_virtual_link[1]" type="continuous">
-      <parent link="finger[${finger_id}]/flex_link[${link_parent}]"/>
-      <child link="finger[${finger_id}]/flex_link[${link_parent}]/virtual_link[1]"/>
-      <origin xyz="${flex_length/num_steps} 0 0" />
-      <axis xyz="0 -1 0"/>
-    </joint>
-    <joint name="finger[${finger_id}]/flex_link[${link_parent}]/flex_joint_from_virtual_link[1]_to_virtual_link[2]" type="continuous">
-      <parent link="finger[${finger_id}]/flex_link[${link_parent}]/virtual_link[1]"/>
-      <child link="finger[${finger_id}]/flex_link[${link_parent}]/virtual_link[2]"/>
-      <origin xyz="0 0 0" />
-      <axis xyz="-1 0 0"/>
-    </joint>
-    <joint name="finger[${finger_id}]/flex_link[${link_parent}]/flex_joint_from_virtual_link[2]_to_flex_link[${link_child}]" type="continuous">
-      <parent link="finger[${finger_id}]/flex_link[${link_parent}]/virtual_link[2]"/>
-      <child link="finger[${finger_id}]/flex_link[${link_child}]"/>
-      <origin xyz="0 0 0" />
-      <axis xyz="0 0 -1"/>
-    </joint>
-  </xacro:macro>
-  <!-- Macro to make the joint from proximal to first link and from last link to distal  -->
-  <xacro:macro name="flex_to_segment_joint" params="finger_id">
-    <link name="finger[${finger_id}]/prox/virtual_link[1]"/>
-    <link name="finger[${finger_id}]/prox/virtual_link[2]"/>
-    <joint name="finger[${finger_id}]/prox/flex_joint_from_prox_to_virtual_link[1]" type="continuous">
-      <parent link="proximal_${finger_id}"/>
-      <child link="finger[${finger_id}]/prox/virtual_link[1]"/>
-      <origin xyz="${prox_length} 0 -0.004"/>
-      <axis xyz="0 -1 0"/>
-    </joint>
-    <joint name="finger[${finger_id}]/prox/flex_joint_from_virtual_link[1]_to_virtual_link[2]" type="continuous">
-      <parent link="finger[${finger_id}]/prox/virtual_link[1]"/>
-      <child link="finger[${finger_id}]/prox/virtual_link[2]"/>
-      <origin xyz="0 0 0"/>
-      <axis xyz="-1 0 0"/>
-    </joint>
-    <joint name="finger[${finger_id}]/prox/flex_joint_from_virtual_link[2]_to_flex_link[1]" type="continuous">
-      <parent link="finger[${finger_id}]/prox/virtual_link[2]"/>
-      <child link="finger[${finger_id}]/flex_link[1]"/>
-      <origin xyz="0 0 0"/>
-      <axis xyz="0 0 -1"/>
-    </joint>
-    <joint name="finger[${finger_id}]/flex_link[${num_steps}]/flex_joint_from_flex_link[${num_steps}]_to_virtual_link[1]" type="continuous">
-      <parent link="finger[${finger_id}]/flex_link[${num_steps}]"/>
-      <child link="finger[${finger_id}]/flex_link[${num_steps}]/virtual_link[1]"/>
-      <origin xyz="${flex_length/num_steps-0.01} 0 0.008"/>
-      <axis xyz="0 -1 0"/>
-    </joint>
-    <joint name="finger[${finger_id}]/flex_link[${num_steps}]/flex_joint_from_virtual_link[1]_to_virtual_link[2]" type="continuous">
-      <parent link="finger[${finger_id}]/flex_link[${num_steps}]/virtual_link[1]"/>
-      <child link="finger[${finger_id}]/flex_link[${num_steps}]/virtual_link[2]"/>
-      <origin xyz="0 0 0"/>
-      <axis xyz="-1 0 0"/>
-    </joint>
-    <joint name="finger[${finger_id}]/flex_link[${num_steps}]/flex_joint_from_virtual_link[2]_to_dist" type="continuous">
-      <parent link="finger[${finger_id}]/flex_link[${num_steps}]/virtual_link[2]"/>
-      <child link="distal_${finger_id}"/>
-      <origin xyz="0 0 0"/>
-      <axis xyz="0 0 -1"/>
-    </joint>
-  </xacro:macro>
-  <xacro:flex_link finger_id="1" flex_id="1"/>
+	<!-- Macro to one flex body link to the next -->
+	<xacro:macro name="flex_joint" params="finger_id link_parent link_child">
+		<joint name="finger[${finger_id}]/flex_joint_from_${link_parent}_to_${link_child}" type="continuous">
+			<parent link="finger[${finger_id}]/flex_link[${link_parent}]"/>
+			<child link="finger[${finger_id}]/flex_link[${link_child}]"/>
+			<origin xyz="${flex_length/num_steps} 0 0" />
+			<axis xyz="0 -1 0"/>
+		</joint>
+	</xacro:macro>
+	<!-- Macro to make the joint from proximal to first link and from last link to distal  -->
+	<xacro:macro name="flex_to_segment_joint" params="finger_id">
+		<joint name="finger[${finger_id}]/flex_joint_from_prox_to_1" type="continuous">
+			<parent link="proximal_${finger_id}"/>
+			<child link="finger[${finger_id}]/flex_link[1]"/>
+			<origin xyz="${prox_length} 0 -0.004"/>
+			<axis xyz="0 -1 0"/>
+		</joint>
+		<joint name="finger[${finger_id}]/flex_joint_from_${num_steps}_to_dist" type="continuous">
+			<parent link="finger[${finger_id}]/flex_link[${num_steps}]"/>
+			<child link="distal_${finger_id}"/>
+			<origin xyz="${flex_length/num_steps-0.01} 0 0.008"/>
+			<axis xyz="0 -1 0"/>
+		</joint>
+	</xacro:macro>
+	<xacro:flex_link finger_id="1" flex_id="1"/>
   <xacro:flex_link finger_id="1" flex_id="2"/>
   <xacro:flex_link finger_id="1" flex_id="3"/>
-  <xacro:flex_link finger_id="1" flex_id="4"/>
+	<xacro:flex_link finger_id="1" flex_id="4"/>
   <xacro:flex_link finger_id="1" flex_id="5"/>
   <xacro:flex_link finger_id="1" flex_id="6"/>
-  <xacro:flex_link finger_id="1" flex_id="7"/>
+ 	<xacro:flex_link finger_id="1" flex_id="7"/>
   <xacro:flex_link finger_id="1" flex_id="8"/>
   <xacro:flex_link finger_id="1" flex_id="9"/>
-  <xacro:flex_joint finger_id="1" link_parent="1" link_child="2"/>
+	<xacro:flex_joint finger_id="1" link_parent="1" link_child="2"/>
   <xacro:flex_joint finger_id="1" link_parent="2" link_child="3"/>
-  <xacro:flex_joint finger_id="1" link_parent="3" link_child="4"/>
+	<xacro:flex_joint finger_id="1" link_parent="3" link_child="4"/>
   <xacro:flex_joint finger_id="1" link_parent="4" link_child="5"/>
-  <xacro:flex_joint finger_id="1" link_parent="5" link_child="6"/>
+	<xacro:flex_joint finger_id="1" link_parent="5" link_child="6"/>
   <xacro:flex_joint finger_id="1" link_parent="6" link_child="7"/>
-  <xacro:flex_joint finger_id="1" link_parent="7" link_child="8"/>
+	<xacro:flex_joint finger_id="1" link_parent="7" link_child="8"/>
   <xacro:flex_joint finger_id="1" link_parent="8" link_child="9"/>
-  <xacro:flex_to_segment_joint finger_id="1"/>
-  <xacro:flex_link finger_id="2" flex_id="1"/>
+ 	<xacro:flex_to_segment_joint finger_id="1"/>
+	<xacro:flex_link finger_id="2" flex_id="1"/>
   <xacro:flex_link finger_id="2" flex_id="2"/>
   <xacro:flex_link finger_id="2" flex_id="3"/>
-  <xacro:flex_link finger_id="2" flex_id="4"/>
+	<xacro:flex_link finger_id="2" flex_id="4"/>
   <xacro:flex_link finger_id="2" flex_id="5"/>
   <xacro:flex_link finger_id="2" flex_id="6"/>
-  <xacro:flex_link finger_id="2" flex_id="7"/>
+ 	<xacro:flex_link finger_id="2" flex_id="7"/>
   <xacro:flex_link finger_id="2" flex_id="8"/>
   <xacro:flex_link finger_id="2" flex_id="9"/>
-  <xacro:flex_joint finger_id="2" link_parent="1" link_child="2"/>
+	<xacro:flex_joint finger_id="2" link_parent="1" link_child="2"/>
   <xacro:flex_joint finger_id="2" link_parent="2" link_child="3"/>
-  <xacro:flex_joint finger_id="2" link_parent="3" link_child="4"/>
+	<xacro:flex_joint finger_id="2" link_parent="3" link_child="4"/>
   <xacro:flex_joint finger_id="2" link_parent="4" link_child="5"/>
-  <xacro:flex_joint finger_id="2" link_parent="5" link_child="6"/>
+	<xacro:flex_joint finger_id="2" link_parent="5" link_child="6"/>
   <xacro:flex_joint finger_id="2" link_parent="6" link_child="7"/>
-  <xacro:flex_joint finger_id="2" link_parent="7" link_child="8"/>
+	<xacro:flex_joint finger_id="2" link_parent="7" link_child="8"/>
   <xacro:flex_joint finger_id="2" link_parent="8" link_child="9"/>
-  <xacro:flex_to_segment_joint finger_id="2"/>
-  <xacro:flex_link finger_id="3" flex_id="1"/>
+ 	<xacro:flex_to_segment_joint finger_id="2"/>
+	<xacro:flex_link finger_id="3" flex_id="1"/>
   <xacro:flex_link finger_id="3" flex_id="2"/>
   <xacro:flex_link finger_id="3" flex_id="3"/>
-  <xacro:flex_link finger_id="3" flex_id="4"/>
+	<xacro:flex_link finger_id="3" flex_id="4"/>
   <xacro:flex_link finger_id="3" flex_id="5"/>
   <xacro:flex_link finger_id="3" flex_id="6"/>
-  <xacro:flex_link finger_id="3" flex_id="7"/>
+ 	<xacro:flex_link finger_id="3" flex_id="7"/>
   <xacro:flex_link finger_id="3" flex_id="8"/>
   <xacro:flex_link finger_id="3" flex_id="9"/>
-  <xacro:flex_joint finger_id="3" link_parent="1" link_child="2"/>
+	<xacro:flex_joint finger_id="3" link_parent="1" link_child="2"/>
   <xacro:flex_joint finger_id="3" link_parent="2" link_child="3"/>
-  <xacro:flex_joint finger_id="3" link_parent="3" link_child="4"/>
+	<xacro:flex_joint finger_id="3" link_parent="3" link_child="4"/>
   <xacro:flex_joint finger_id="3" link_parent="4" link_child="5"/>
-  <xacro:flex_joint finger_id="3" link_parent="5" link_child="6"/>
+	<xacro:flex_joint finger_id="3" link_parent="5" link_child="6"/>
   <xacro:flex_joint finger_id="3" link_parent="6" link_child="7"/>
-  <xacro:flex_joint finger_id="3" link_parent="7" link_child="8"/>
+	<xacro:flex_joint finger_id="3" link_parent="7" link_child="8"/>
   <xacro:flex_joint finger_id="3" link_parent="8" link_child="9"/>
-  <xacro:flex_to_segment_joint finger_id="3"/>
+ 	<xacro:flex_to_segment_joint finger_id="3"/>
 <!-- ################ ################ ################ ################ ################ ################ -->
 <!-- ################ THE SECTION CREATED BY SOLIDWORKS EXPORTER, CUT AND PASTE THIS IN HERE ################ -->
@@ -263,5 +223,5 @@
     <origin
       xyz="0.01 0 0.0186"
-      rpy="-6.20039667432211E-16 0.05 2.22044604925031E-16" />
+      rpy="-6.20039667432211E-16 0 2.22044604925031E-16" />
     <parent
       link="swivel_1" />
@@ -408,5 +368,5 @@
     <origin
       xyz="0.01 0 0.0186"
-      rpy="-1.16908225836102E-15 0.05 1.11022302462515E-16" />
+      rpy="-1.16908225836102E-15 0 1.11022302462515E-16" />
     <parent
       link="swivel_2" />
@@ -524,5 +484,5 @@
     <origin
       xyz="-0.0299999999999996 0 0.0816000000000002"
-      rpy="-5.55111512312578E-17 0.05 3.14159265358979" />
+      rpy="-5.55111512312578E-17 0 3.14159265358979" />
     <parent
       link="base_link" />
