Commit message: macroified the hand model to support multiple girppers

File: reflex_visualizer/urdf/full_reflex_model.urdf.xacro (robot description, xacro)
@@ -1,4 +1,6 @@
 <?xml version="1.0"?>
-<robot xmlns:xacro="http://www.ros.org/wiki/xacro" name="rhr_flex_model">
+<robot xmlns:xacro="http://www.ros.org/wiki/xacro" name="${tf_prefix}rhr_flex_model">
+	<xacro:arg name="attached" default="true"/>
+	<xacro:property name="has_parent" value="$(arg attached)"/>
 <!-- ################ ################ ################ ################ ################ ################ -->
 <!-- ################ XACRO PORTION OF THE URDF, FOR MAKING THE FLEXIBLE JOINTS ################ -->
@@ -29,5 +31,5 @@
   <xacro:macro name="flex_link" params="finger_id flex_id">
     <link
-      name="finger[${finger_id}]/flex_link[${flex_id}]">
+      name="${tf_prefix}finger[${finger_id}]/flex_link[${flex_id}]">
       <visual>
         <origin
@@ -39,5 +41,5 @@
         </geometry>
         <material
-          name="">
+          name="${tf_prefix}">
           <xacro:flex_color/>
         </material>
@@ -47,7 +49,7 @@
 	<!-- Macro to one flex body link to the next -->
 	<xacro:macro name="flex_joint" params="finger_id link_parent link_child">
-		<joint name="finger[${finger_id}]/flex_joint_from_${link_parent}_to_${link_child}" type="continuous">
-			<parent link="finger[${finger_id}]/flex_link[${link_parent}]"/>
-			<child link="finger[${finger_id}]/flex_link[${link_child}]"/>
+		<joint name="${tf_prefix}finger[${finger_id}]/flex_joint_from_${link_parent}_to_${link_child}" type="continuous">
+			<parent link="${tf_prefix}finger[${finger_id}]/flex_link[${link_parent}]"/>
+			<child link="${tf_prefix}finger[${finger_id}]/flex_link[${link_child}]"/>
 			<origin xyz="${flex_length/num_steps} 0 0" />
 			<axis xyz="0 -1 0"/>
@@ -56,71 +58,79 @@
 	<!-- Macro to make the joint from proximal to first link and from last link to distal  -->
 	<xacro:macro name="flex_to_segment_joint" params="finger_id">
-		<joint name="finger[${finger_id}]/flex_joint_from_prox_to_1" type="continuous">
-			<parent link="proximal_${finger_id}"/>
-			<child link="finger[${finger_id}]/flex_link[1]"/>
+		<joint name="${tf_prefix}finger[${finger_id}]/flex_joint_from_prox_to_1" type="continuous">
+			<parent link="${tf_prefix}proximal_${finger_id}"/>
+			<child link="${tf_prefix}finger[${finger_id}]/flex_link[1]"/>
 			<origin xyz="${prox_length} 0 -0.004"/>
 			<axis xyz="0 -1 0"/>
 		</joint>
-		<joint name="finger[${finger_id}]/flex_joint_from_${num_steps}_to_dist" type="continuous">
-			<parent link="finger[${finger_id}]/flex_link[${num_steps}]"/>
-			<child link="distal_${finger_id}"/>
+		<joint name="${tf_prefix}finger[${finger_id}]/flex_joint_from_${num_steps}_to_dist" type="continuous">
+			<parent link="${tf_prefix}finger[${finger_id}]/flex_link[${num_steps}]"/>
+			<child link="${tf_prefix}distal_${finger_id}"/>
 			<origin xyz="${flex_length/num_steps-0.01} 0 0.008"/>
 			<axis xyz="0 -1 0"/>
 		</joint>
 	</xacro:macro>
-	<xacro:flex_link finger_id="1" flex_id="1"/>
-  <xacro:flex_link finger_id="1" flex_id="2"/>
-  <xacro:flex_link finger_id="1" flex_id="3"/>
-	<xacro:flex_link finger_id="1" flex_id="4"/>
-  <xacro:flex_link finger_id="1" flex_id="5"/>
-  <xacro:flex_link finger_id="1" flex_id="6"/>
- 	<xacro:flex_link finger_id="1" flex_id="7"/>
-  <xacro:flex_link finger_id="1" flex_id="8"/>
-  <xacro:flex_link finger_id="1" flex_id="9"/>
-	<xacro:flex_joint finger_id="1" link_parent="1" link_child="2"/>
-  <xacro:flex_joint finger_id="1" link_parent="2" link_child="3"/>
-	<xacro:flex_joint finger_id="1" link_parent="3" link_child="4"/>
-  <xacro:flex_joint finger_id="1" link_parent="4" link_child="5"/>
-	<xacro:flex_joint finger_id="1" link_parent="5" link_child="6"/>
-  <xacro:flex_joint finger_id="1" link_parent="6" link_child="7"/>
-	<xacro:flex_joint finger_id="1" link_parent="7" link_child="8"/>
-  <xacro:flex_joint finger_id="1" link_parent="8" link_child="9"/>
- 	<xacro:flex_to_segment_joint finger_id="1"/>
-	<xacro:flex_link finger_id="2" flex_id="1"/>
-  <xacro:flex_link finger_id="2" flex_id="2"/>
-  <xacro:flex_link finger_id="2" flex_id="3"/>
-	<xacro:flex_link finger_id="2" flex_id="4"/>
-  <xacro:flex_link finger_id="2" flex_id="5"/>
-  <xacro:flex_link finger_id="2" flex_id="6"/>
- 	<xacro:flex_link finger_id="2" flex_id="7"/>
-  <xacro:flex_link finger_id="2" flex_id="8"/>
-  <xacro:flex_link finger_id="2" flex_id="9"/>
-	<xacro:flex_joint finger_id="2" link_parent="1" link_child="2"/>
-  <xacro:flex_joint finger_id="2" link_parent="2" link_child="3"/>
-	<xacro:flex_joint finger_id="2" link_parent="3" link_child="4"/>
-  <xacro:flex_joint finger_id="2" link_parent="4" link_child="5"/>
-	<xacro:flex_joint finger_id="2" link_parent="5" link_child="6"/>
-  <xacro:flex_joint finger_id="2" link_parent="6" link_child="7"/>
-	<xacro:flex_joint finger_id="2" link_parent="7" link_child="8"/>
-  <xacro:flex_joint finger_id="2" link_parent="8" link_child="9"/>
- 	<xacro:flex_to_segment_joint finger_id="2"/>
-	<xacro:flex_link finger_id="3" flex_id="1"/>
-  <xacro:flex_link finger_id="3" flex_id="2"/>
-  <xacro:flex_link finger_id="3" flex_id="3"/>
-	<xacro:flex_link finger_id="3" flex_id="4"/>
-  <xacro:flex_link finger_id="3" flex_id="5"/>
-  <xacro:flex_link finger_id="3" flex_id="6"/>
- 	<xacro:flex_link finger_id="3" flex_id="7"/>
-  <xacro:flex_link finger_id="3" flex_id="8"/>
-  <xacro:flex_link finger_id="3" flex_id="9"/>
-	<xacro:flex_joint finger_id="3" link_parent="1" link_child="2"/>
-  <xacro:flex_joint finger_id="3" link_parent="2" link_child="3"/>
-	<xacro:flex_joint finger_id="3" link_parent="3" link_child="4"/>
-  <xacro:flex_joint finger_id="3" link_parent="4" link_child="5"/>
-	<xacro:flex_joint finger_id="3" link_parent="5" link_child="6"/>
-  <xacro:flex_joint finger_id="3" link_parent="6" link_child="7"/>
-	<xacro:flex_joint finger_id="3" link_parent="7" link_child="8"/>
-  <xacro:flex_joint finger_id="3" link_parent="8" link_child="9"/>
- 	<xacro:flex_to_segment_joint finger_id="3"/>
+	<xacro:macro name="reflex_xacro" params="tf_prefix='' parent='' *origin">
+		<xacro:flex_link finger_id="1" flex_id="1"/>
+	  <xacro:flex_link finger_id="1" flex_id="2"/>
+	  <xacro:flex_link finger_id="1" flex_id="3"/>
+		<xacro:flex_link finger_id="1" flex_id="4"/>
+	  <xacro:flex_link finger_id="1" flex_id="5"/>
+	  <xacro:flex_link finger_id="1" flex_id="6"/>
+	 	<xacro:flex_link finger_id="1" flex_id="7"/>
+	  <xacro:flex_link finger_id="1" flex_id="8"/>
+	  <xacro:flex_link finger_id="1" flex_id="9"/>
+		<xacro:flex_joint finger_id="1" link_parent="1" link_child="2"/>
+	  <xacro:flex_joint finger_id="1" link_parent="2" link_child="3"/>
+		<xacro:flex_joint finger_id="1" link_parent="3" link_child="4"/>
+	  <xacro:flex_joint finger_id="1" link_parent="4" link_child="5"/>
+		<xacro:flex_joint finger_id="1" link_parent="5" link_child="6"/>
+	  <xacro:flex_joint finger_id="1" link_parent="6" link_child="7"/>
+		<xacro:flex_joint finger_id="1" link_parent="7" link_child="8"/>
+	  <xacro:flex_joint finger_id="1" link_parent="8" link_child="9"/>
+	 	<xacro:flex_to_segment_joint finger_id="1"/>
+		<xacro:flex_link finger_id="2" flex_id="1"/>
+	  <xacro:flex_link finger_id="2" flex_id="2"/>
+	  <xacro:flex_link finger_id="2" flex_id="3"/>
+		<xacro:flex_link finger_id="2" flex_id="4"/>
+	  <xacro:flex_link finger_id="2" flex_id="5"/>
+	  <xacro:flex_link finger_id="2" flex_id="6"/>
+	 	<xacro:flex_link finger_id="2" flex_id="7"/>
+	  <xacro:flex_link finger_id="2" flex_id="8"/>
+	  <xacro:flex_link finger_id="2" flex_id="9"/>
+		<xacro:flex_joint finger_id="2" link_parent="1" link_child="2"/>
+	  <xacro:flex_joint finger_id="2" link_parent="2" link_child="3"/>
+		<xacro:flex_joint finger_id="2" link_parent="3" link_child="4"/>
+	  <xacro:flex_joint finger_id="2" link_parent="4" link_child="5"/>
+		<xacro:flex_joint finger_id="2" link_parent="5" link_child="6"/>
+	  <xacro:flex_joint finger_id="2" link_parent="6" link_child="7"/>
+		<xacro:flex_joint finger_id="2" link_parent="7" link_child="8"/>
+	  <xacro:flex_joint finger_id="2" link_parent="8" link_child="9"/>
+	 	<xacro:flex_to_segment_joint finger_id="2"/>
+		<xacro:flex_link finger_id="3" flex_id="1"/>
+	  <xacro:flex_link finger_id="3" flex_id="2"/>
+	  <xacro:flex_link finger_id="3" flex_id="3"/>
+		<xacro:flex_link finger_id="3" flex_id="4"/>
+	  <xacro:flex_link finger_id="3" flex_id="5"/>
+	  <xacro:flex_link finger_id="3" flex_id="6"/>
+	 	<xacro:flex_link finger_id="3" flex_id="7"/>
+	  <xacro:flex_link finger_id="3" flex_id="8"/>
+	  <xacro:flex_link finger_id="3" flex_id="9"/>
+		<xacro:flex_joint finger_id="3" link_parent="1" link_child="2"/>
+	  <xacro:flex_joint finger_id="3" link_parent="2" link_child="3"/>
+		<xacro:flex_joint finger_id="3" link_parent="3" link_child="4"/>
+	  <xacro:flex_joint finger_id="3" link_parent="4" link_child="5"/>
+		<xacro:flex_joint finger_id="3" link_parent="5" link_child="6"/>
+	  <xacro:flex_joint finger_id="3" link_parent="6" link_child="7"/>
+		<xacro:flex_joint finger_id="3" link_parent="7" link_child="8"/>
+	  <xacro:flex_joint finger_id="3" link_parent="8" link_child="9"/>
+	 	<xacro:flex_to_segment_joint finger_id="3"/>
+		<xacro:if value="${has_parent}">
+			<joint name="${tf_prefix}_to_hand_joint" type="fixed">
+				<xacro:insert_block name="origin"/>
+				<parent link="${parent}"/>
+				<child link="${tf_prefix}hand_base"/>
+			</joint>
+		</xacro:if>
 <!-- ################ ################ ################ ################ ################ ################ -->
 <!-- ################ THE SECTION CREATED BY SOLIDWORKS EXPORTER, CUT AND PASTE THIS IN HERE ################ -->
@@ -128,500 +138,501 @@
 <!-- ################ COMMENT OUT ALL dist*_joint PIECES OF THIS URDF SO THE FLEX JOINTS CAN LINK UP ################ -->
 <!-- ################ ################ ################ ################ ################ ################ -->
-  <link
-    name="base_link">
-    <visual>
-      <origin
-        xyz="0 0 0"
-        rpy="0 0 0" />
-      <geometry>
-        <mesh
-          filename="package://reflex_visualizer/meshes/base_link.STL" />
-      </geometry>
-      <material
-        name="">
-        <xacro:base_color/>
-      </material>
-    </visual>
-  </link>
-  <link
-    name="pad">
-    <visual>
-      <origin
-        xyz="0 0 0"
-        rpy="0 0 0" />
-      <geometry>
-        <mesh
-          filename="package://reflex_visualizer/meshes/pad.STL" />
-      </geometry>
-      <material
-        name="">
-        <xacro:pad_color/>
-      </material>
-    </visual>
-  </link>
-  <joint
-    name="pad_joint"
-    type="fixed">
-    <origin
-      xyz="0.02 0 0.063"
-      rpy="1.5707963267949 5.55111512312578E-17 -1.5707963267949" />
-    <parent
-      link="base_link" />
-    <child
-      link="pad" />
-    <axis
-      xyz="0 0 0" />
-  </joint>
-  <link
-    name="swivel_1">
-    <visual>
-      <origin
-        xyz="0 0 0"
-        rpy="0 0 0" />
-      <geometry>
-        <mesh
-          filename="package://reflex_visualizer/meshes/swivel_1.STL" />
-      </geometry>
-      <material
-        name="">
-        <xacro:swivel_color/>
-      </material>
-    </visual>
-  </link>
-  <joint
-    name="preshape_1"
-    type="continuous">
-    <origin
-      xyz="0.0503973683071414 -0.026 0.063"
-      rpy="6.75550818663469E-16 1.97993848419069E-16 -2.77555756156289E-16" />
-    <parent
-      link="base_link" />
-    <child
-      link="swivel_1" />
-    <axis
-      xyz="0 0 -1" />
-  </joint>
-  <link
-    name="proximal_1">
-    <visual>
-      <origin
-        xyz="-0.011 0.007 0.011"
-        rpy="3.1459 0 0"/>
-      <geometry>
-        <mesh
-          filename="package://reflex_visualizer/meshes/proximal_1.STL" />
-      </geometry>
-      <material
-        name="">
-        <xacro:proximal_color/>
-      </material>
-    </visual>
-  </link>
-  <joint
-    name="proximal_joint_1"
-    type="continuous">
-    <origin
-      xyz="0.01 0 0.0186"
-      rpy="-6.20039667432211E-16 0 2.22044604925031E-16" />
-    <parent
-      link="swivel_1" />
-    <child
-      link="proximal_1" />
-    <axis
-      xyz="0 -1 0" />
-  </joint>
-  <link
-    name="proximal_pad_1">
-    <visual>
-      <origin
-        xyz="-0.008 0.014 -0.002"
-        rpy="1.5708 1.5708 0" />
-      <geometry>
-        <mesh
-          filename="package://reflex_visualizer/meshes/proximal_pad_1.STL" />
-      </geometry>
-      <material
-        name="">
-        <xacro:pad_color/>
-      </material>
-    </visual>
-  </link>
-  <joint
-    name="prox1_pad_joint"
-    type="fixed">
-    <origin
-      xyz="0 0 0"
-      rpy="1.5707963267949 0 -1.5707963267949" />
-    <parent
-      link="proximal_1" />
-    <child
-      link="proximal_pad_1" />
-    <axis
-      xyz="0 0 0" />
-  </joint>
-  <link
-    name="distal_1">
-    <visual>
-      <origin
-        xyz="-0.077 0.007 0.007"
-        rpy="3.1459 0 0" />
-      <geometry>
-        <mesh
-          filename="package://reflex_visualizer/meshes/distal_1.STL" />
-      </geometry>
-      <material
-        name="">
-        <xacro:distal_color/>
-      </material>
-    </visual>
-  </link>
-  <joint
-    name="distal_joint_1"
-    type="continuous">
-    <origin
-      xyz="0.07600000000000001 0 0.00250000000000002"
-      rpy="0 0 0" />
-    <parent
-      link="proximal_1" />
-    <child
-      link="distal_1" />
-    <axis
-      xyz="0 -1 0" />
-  </joint>
-  <link
-    name="distal_pad_1">
-    <visual>
-      <origin
-        xyz="-0.00825 0.009 0.057"
-        rpy="1.5708 1.5708 0" />
-      <geometry>
-        <mesh
-          filename="package://reflex_visualizer/meshes/distal_pad_1.STL" />
-      </geometry>
-      <material
-        name="">
-        <xacro:pad_color/>
-      </material>
-    </visual>
-  </link>
-  <joint
-    name="dist1_pad_joint"
-    type="fixed">
-    <origin
-      xyz="-0.01 0 0.001"
-      rpy="1.5707963267949 0 -1.5707963267949" />
-    <parent
-      link="distal_1" />
-    <child
-      link="distal_pad_1" />
-    <axis
-      xyz="0 0 0" />
-  </joint>
-  <link
-    name="swivel_2">
-    <visual>
-      <origin
-        xyz="0 0 0"
-        rpy="0 0 0" />
-      <geometry>
-        <mesh
-          filename="package://reflex_visualizer/meshes/swivel_2.STL" />
-      </geometry>
-      <material
-        name="">
-        <xacro:swivel_color/>
-      </material>
-    </visual>
-  </link>
-  <joint
-    name="preshape_2"
-    type="continuous">
-    <origin
-      xyz="0.0503973683071413 0.0259999999999999 0.063"
-      rpy="1.22459340959228E-15 -7.33448407631817E-16 -1.66533453693773E-16" />
-    <parent
-      link="base_link" />
-    <child
-      link="swivel_2" />
-    <axis
-      xyz="0 0 -1" />
-  </joint>
-  <link
-    name="proximal_2">
-    <visual>
-      <origin
-        xyz="-0.011 0.007 0.011"
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
Commit message: small change of parent params

File: reflex_visualizer/urdf/full_reflex_model.urdf.xacro (robot description, xacro)
@@ -71,5 +71,5 @@
 		</joint>
 	</xacro:macro>
-	<xacro:macro name="reflex_xacro" params="tf_prefix='' parent='' *origin">
+	<xacro:macro name="reflex_xacro" params="tf_prefix='' parent='' twist=0">
 		<xacro:flex_link finger_id="1" flex_id="1"/>
 	  <xacro:flex_link finger_id="1" flex_id="2"/>
@@ -127,6 +127,6 @@
 	 	<xacro:flex_to_segment_joint finger_id="3"/>
 		<xacro:if value="${has_parent}">
-			<joint name="${tf_prefix}_to_hand_joint" type="fixed">
-				<xacro:insert_block name="origin"/>
+			<joint name="${tf_prefix}to_hand_joint" type="fixed">
+				<origin rpy="0 0 ${twist}" xyz="0 0 0"/>
 				<parent link="${parent}"/>
 				<child link="${tf_prefix}hand_base"/>
